File: 40split2/40split2.kicad_pcb (KiCad board)
At the start: 2 copper layers, 145.3 x 97 mm, 47 parts

Commit message: Fixed a bunch of errors, added more plans
Parts:
- removed the REF** at (101.2, 136.9)
- added REF**: SolderJumper-2_P1.3mm_Open_Pad1.0x1.5mm, rp2040-zero:SolderJumper-2_P1.3mm_Open_Pad1.0x1.5mm, F.Cu at (199.8, 70.5)
- added REF**: SolderJumper-2_P1.3mm_Open_Pad1.0x1.5mm, rp2040-zero:SolderJumper-2_P1.3mm_Open_Pad1.0x1.5mm, F.Cu at (199.8, 66.7)
- added REF**: SolderJumper-2_P1.3mm_Open_Pad1.0x1.5mm, rp2040-zero:SolderJumper-2_P1.3mm_Open_Pad1.0x1.5mm, B.Cu at (199.8, 66.7)
- added REF**: SolderJumper-2_P1.3mm_Open_Pad1.0x1.5mm, rp2040-zero:SolderJumper-2_P1.3mm_Open_Pad1.0x1.5mm, B.Cu at (199.8, 70.5)
- moved REF** 26.2 mm to (108.1, 130.5)
- moved REF** 0.82 mm to (213.8, 66.5)
- moved U 0.31 mm to (199.8, 74.7)
Routing:
- net (no net): track 0.00 -> 4021.3 mm, vias 0 -> 32
Other:
- outline, holes or cut-outs redrawn

Commit message: new diode cluster
Parts:
- removed the REF** at (121.9, 134.3)
- removed the REF** at (127.5, 131.9)
- removed the REF** at (131.1, 136.9)
- removed the REF** at (132.1, 133.2)
- removed the REF** at (118.4, 129.4)
- removed the REF** at (125.2, 131.3)
- removed the REF** at (129.8, 132.5)
- removed the REF** at (124.2, 134.9)
- removed the REF** at (117.3, 133.0)
- removed the REF** at (128.8, 136.2)
- removed the REF** at (111.5, 127.4)
- removed the REF** at (113.8, 128.1)
- removed the REF** at (120.7, 130.0)
- removed the REF** at (126.5, 135.6)
- removed the REF** at (123.0, 130.6)
- removed the REF** at (134.4, 133.8)
- removed the REF** at (112.8, 131.8)
- removed the REF** at (108.1, 130.5)
- removed the REF** at (115.0, 132.4)
- removed the REF** at (116.1, 128.7)
- removed the REF** at (110.5, 131.1)
- removed the REF** at (119.6, 133.7)
- added REF**: 1N4148, Scotto_lib:Diode_DO-35, F.Cu at (121.8, 134.7)
- added REF**: 1N4148, Scotto_lib:Diode_DO-35, F.Cu at (131.5, 137.4)
- added REF**: 1N4148, Scotto_lib:Diode_DO-35, F.Cu at (143.2, 119.9)
- added REF**: 1N4148, Scotto_lib:Diode_DO-35, F.Cu at (151.8, 141.5)
- added REF**: 1N4148, Scotto_lib:Diode_DO-35, F.Cu at (123.5, 129.0)
- added REF**: 1N4148, Scotto_lib:Diode_DO-35, F.Cu at (112.2, 132.0)
- added REF**: 1N4148, Scotto_lib:Diode_DO-35, F.Cu at (122.7, 131.8)
- added REF**: 1N4148, Scotto_lib:Diode_DO-35, F.Cu at (120.9, 122.0)
- added REF**: 1N4148, Scotto_lib:Diode_DO-35, F.Cu at (133.1, 131.6)
- added REF**: 1N4148, Scotto_lib:Diode_DO-35, F.Cu at (124.3, 126.1)
- added REF**: 1N4148, Scotto_lib:Diode_DO-35, F.Cu at (113.0, 129.2)
- added REF**: 1N4148, Scotto_lib:Diode_DO-35, F.Cu at (113.8, 126.3)
- added REF**: 1N4148, Scotto_lib:Diode_DO-35, F.Cu at (133.9, 128.8)
- added REF**: 1N4148, Scotto_lib:Diode_DO-35, F.Cu at (133.1, 116.1)
- added REF**: 1N4148, Scotto_lib:Diode_DO-35, F.Cu at (141.7, 138.8)
- added REF**: 1N4148, Scotto_lib:Diode_DO-35, F.Cu at (103.2, 126.4)
- added REF**: 1N4148, Scotto_lib:Diode_DO-35, F.Cu at (131.5, 121.8)
- added REF**: 1N4148, Scotto_lib:Diode_DO-35, F.Cu at (102.4, 129.3)
- added REF**: 1N4148, Scotto_lib:Diode_DO-35, F.Cu at (130.7, 124.7)
- added REF**: 1N4148, Scotto_lib:Diode_DO-35, F.Cu at (132.3, 119.0)
- added REF**: 1N4148, Scotto_lib:Diode_DO-35, F.Cu at (132.3, 134.5)
- added REF**: 1N4148, Scotto_lib:Diode_DO-35, F.Cu at (114.6, 123.4)
Routing:
- net (no net): track 4021.3 -> 3853.1 mm, vias 32 -> 10
