File: 40split2/_autosave-40split2.kicad_pcb (KiCad board)
At the start: 2 copper layers, 145.3 x 97 mm, 54 parts

Commit message: make some changes to the pcb
Other:
- board text added: ":3"
- board text added: "Bridge these if they are on the TOP"
- board text added: "github.com/junnnaaaaaa github.com/HamNuggets"
Changed lines of the file:
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@@
 			(at 0 1.8 90)
 			(layer "B.SilkS")
+			(hide yes)
 			(effects
 				(font
@@
 			(at 0 1.8 90)
 			(layer "B.SilkS")
+			(hide yes)
 			(effects
 				(font
@@
 		(layer "Edge.Cuts")
 	)
+	(gr_text "Bridge these if\nthey are on the\nTOP"
+		(at 193.99 80.27 0)
+		(layer "F.SilkS")
+		(effects
+			(font
+				(size 1 1)
+				(thickness 0.1)
+			)
+			(justify left bottom)
+		)
+	)
+	(gr_text ":3"
+		(at 189.19 150.27 0)
+		(layer "F.SilkS")
+		(effects
+			(font
+				(size 4 4)
+				(thickness 0.4)
+			)
+			(justify left bottom)
+		)
+	)
+	(gr_text "Bridge these if\nthey are on the\nTOP"
+		(at 205.79 80.27 -0)
+		(layer "B.SilkS")
+		(effects
+			(font
+				(size 1 1)
+				(thickness 0.1)
+			)
+			(justify left bottom mirror)
+		)
+	)
+	(gr_text ":3"
+		(at 195.19 150.27 -0)
+		(layer "B.SilkS")
+		(effects
+			(font
+				(size 4 4)
+				(thickness 0.4)
+			)
+			(justify left bottom mirror)
+		)
+	)
+	(gr_text "github.com/junnnaaaaaa\ngithub.com/HamNuggets"
+		(at 184.59 83.67 0)
+		(layer "B.SilkS")
+		(effects
+			(font
+				(size 0.5 0.5)
+				(thickness 0.0625)
+			)
+			(justify left bottom mirror)
+		)
+	)
 	(segment
